File: valve_controller_v1/usb.kicad_sch (KiCad schematic)
At the start: 9 parts, among them J4 USB_C_Receptacle_USB2.0_16P, U3 CH340E

Commit message: Assigned footprints
Assigned footprints
Selected JLCPCB part numbers and searched for alternatives for some components (diodes, transistors)
Imported previos footprint library
Parts:
- J4: JLCPCB (none) -> C319148
- U3: JLCPCB (none) -> C99652
Changed lines of the file:
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@@
+			)
+		)
+		(property "JLCPCB" "C319148"
+			(at 40.64 63.5 0)
+			(effects
+				(font
+					(size 0.762 0.762)
+					(italic yes)
+				)
 			)
 		)
@@
 		)
 		(property "Value" "CH340E"
-			(at 116.84 66.04 0)
+			(at 115.57 36.83 0)
 			(effects
 				(font
@@
 			)
 		)
+		(property "JLCPCB" "C99652"
+			(at 118.11 64.77 0)
+			(effects
+				(font
+					(size 0.762 0.762)
+					(italic yes)
+				)
+			)
+		)
