File: valve_controller_v1/usb.kicad_sch (KiCad schematic)
At the start: 9 parts, among them J4 USB_C_Receptacle_USB2.0_16P, U3 CH340E

Commit message: Final corrections for manufacturing
Created new condenser footprint to better represent the actual position
Created new voltage selector ip switch footprint
Selected bigger footprint for R19 (was 1206 now is 2512 as in the legacy version)
Corrected D5 footprint (was SOD-123 now is SMA)
Parts:
- TP7, TP8: now left out of the parts list
Changed lines of the file:
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@@
 		(unit 1)
 		(exclude_from_sim no)
-		(in_bom yes)
+		(in_bom no)
 		(on_board yes)
 		(dnp no)
@@
 		(unit 1)
 		(exclude_from_sim no)
-		(in_bom yes)
-		(on_board yes)
-		(dnp no)
+		(in_bom no)
+		(on_board yes)
+		(dnp no)
