File: valve_controller_v1/valve-controller_v1.0.kicad_sch (KiCad schematic)
At the start: 72 parts, among them J1 Solar Panel, J2 USB_C_Receptacle_USB2.0_16P, J3 Solenoid Output, J4 Debug & Program, Q1 DMG3415UQ-7, Q2 DMG3415UQ-7, SW1 XKB5858, SW2 Reset, SW3 Boot Selector, SW4 Voltage Selector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

Commit message: Finished first version of the schematic
Added hierarchical sheets for every block (Power, USB, Valve Drivers, MCU, Step Up)
Updated the battery voltage measurement circuit
Assigned footprint for most of the components (Work in Progress)
Placed most of the components near related main active components
Parts:
- removed C1, C11, C2, C3, C4, C7, C9: 10u, symbol Device:C_Small
- removed C10: 220p, symbol Device:C_Small
- removed C12: 4700u, symbol Device:C_Polarized_Small
- removed C13, C5, C6, C8: 100n, symbol Device:C_Small
- removed D1, D2, D3: BS819W, symbol Device:D_Schottky_Small
- removed D4: Yellow, symbol Device:LED_Small_Filled
- removed D5: SS34, symbol Device:D_Schottky_Small
- removed J2: USB_C_Receptacle_USB2.0_16P, symbol Connector:USB_C_Receptacle_USB2.0_16P
- removed J4: Debug & Program, Connector:Tag-Connect_TC2030-IDC-NL_2x03_P1.27mm_Vertical, symbol Connector:Conn_ARM_SWD_TagConnect_TC2030-NL
- removed JP1: VCC_Prog, symbol Jumper:Jumper_2_Small_Open
- removed L1: L_Small, symbol Device:L_Small
- removed Q1, Q2: DMG3415UQ-7, symbol Transistor_FET:Q_PMOS_GSD
- removed R1, R10, R11, R14, R2, R4, R5: 10k, symbol Device:R_Small
- removed R12, R6: 1M, symbol Device:R_Small
- removed R13: 1k, symbol Device:R_Small
- removed R15: 174k, symbol Device:R_Small
- removed R16: 95.3k, symbol Device:R_Small
- removed R17: 243k, symbol Device:R_Small
- removed R18: 34, symbol Device:R_Small
- removed R19, R20: 1.5k, symbol Device:R_Small
- removed R3: 2.7k, symbol Device:R_Small
- removed R7: 1.5M, symbol Device:R_Small
- removed R8, R9: 5.1k, symbol Device:R_Small
- removed SW1: XKB5858, symbol Wisflow:XKB5858-X-F-75
- removed SW2: Reset, symbol Switch:SW_SPST
- removed SW3: Boot Selector, symbol Switch:SW_SPDT
- removed SW4: Voltage Selector, symbol Switch:SW_DIP_x02
- removed TP1: TX, symbol Connector:TestPoint
- removed TP2: RX, symbol Connector:TestPoint
- removed TP3: ~{BAT_MON_EN}, symbol Connector:TestPoint
- removed TP4: BAT_MON, symbol Connector:TestPoint
- removed TP5: REG_EN, symbol Connector:TestPoint
- removed TP6: 3V3, symbol Connector:TestPoint
- removed TP7: V_{CC}, symbol Connector:TestPoint
- removed TP8: V_{BAT}, symbol Connector:TestPoint
- removed U1: XC6220B331MR, Package_TO_SOT_SMD:SOT-23-5, symbol Regulator_Linear:XC6220B331MR
- removed U2: BQ21040DBV, Package_TO_SOT_SMD:SOT-23-6, symbol Battery_Management:BQ21040DBV
- removed U3: CH340E, Package_SO:MSOP-10_3x3mm_P0.5mm, symbol Interface_USB:CH340E
- removed U4: RAK3172-xx-9-SM-xI, RF_Module:RAK3172, symbol RF_Module:RAK3172-xx-9-SM-xI
- removed U5: LMR62421XMF, Package_TO_SOT_SMD:SOT-23-5, symbol Regulator_Switching:LMR62421XMF
- removed U6: LT218, symbol Wisflow:LT218
- removed U7, U8: DRV8231ADSG, Package_SON:WSON-8-1EP_2x2mm_P0.5mm_EP0.9x1.6mm, symbol Driver_Motor:DRV8231ADSG
- removed U9: DRV8845, symbol Wisflow:DRV8845
- added J3: Solenoid #3,4 Output, Connector_Phoenix_MSTB:PhoenixContact_MSTBA_2,5_4-G-5,08_1x04_P5.08mm_Horizontal, symbol Connector_Generic:Conn_01x04
- added J6: Debug, Connector_PinHeader_2.54mm:PinHeader_1x02_P2.54mm_Vertical, symbol Connector_Generic:Conn_01x02
- H1, H2, H3, H4: footprint (none) -> MountingHole:MountingHole_2.2mm_M2
- J1: footprint (none) -> Diode_SMD:D_SMA
- J2: renamed from J3; value Solenoid Output -> Solenoid #1,2 Output; footprint (none) -> Connector_Phoenix_MSTB:PhoenixContact_MSTBA_2,5_4-G-5,08_1x04_P5.08mm_Horizontal
Connections:
- net Valve Driver/S2_O1: now reaches J2.3 (Pin_3)
- net Valve Driver/S2_O2: now reaches J2.4 (Pin_4)
- net S1_O1 renamed Valve Driver/S1_O1
- net S1_O2 renamed Valve Driver/S1_O2
- new net MCU/RAK_DBG_RX: J6.2 (Pin_2)
- new net MCU/RAK_DBG_TX: J6.1 (Pin_1)
- new net Valve Driver/S3_O1: J3.1 (Pin_1)
- new net Valve Driver/S3_O2: J3.2 (Pin_2)
- new net Valve Driver/S4_O1: J3.3 (Pin_3)
- new net Valve Driver/S4_O2: J3.4 (Pin_4)
- no-connect marks 11 -> 0
Other:
- added sheet MCU (mcu.kicad_sch)
- added sheet Power (power.kicad_sch)
- added sheet StepUp (step_up.kicad_sch)
- added sheet USB (usb.kicad_sch)
- added sheet Valve Driver (valve_driver.kicad_sch)
- note added: "Main Power Inputs"
- note removed: "Battery charger"
- note removed: "Battery charger and Solar panel"
- note removed: "Battery monitor"
- note removed: "Inverse polarity protection"
- note removed: "JLCPCB: C780036"
- note removed: "Power Input"
- note removed: "Revisar este circuito Como se puede apagar, se pueden usar resistencias mas chicas que dan una mejor medida"
- note removed: "USB & UART"
- note removed: "USB to UART"
- note removed: "Voltage regulator & Power switch"
- moved on the sheet: BT1, H1, H2, H3, H4, J1, J2

Commit message: Assigned footprints
Assigned footprints
Selected JLCPCB part numbers and searched for alternatives for some components (diodes, transistors)
Imported previos footprint library
Parts:
- BT1: footprint (none) -> Wisflow:BatteryHolder_MPD_BK-18650-PC2; JLCPCB (none) -> C19184084
- J1: footprint Diode_SMD:D_SMA -> Connector_JST:JST_EH_S2B-EH_1x02_P2.50mm_Horizontal
- J2, J3: now left out of the parts list
- J6: footprint Connector_PinHeader_2.54mm:PinHeader_1x02_P2.54mm_Vertical -> Connector_PinHeader_2.54mm:PinHeader_1x03_P2.54mm_Vertical; symbol Connector_Generic:Conn_01x02 -> Connector_Generic:Conn_01x03
Connections:
- net GND: now also J6.3 (Pin_3)
Other:
- note added: "DNP"
Changed lines of the file:
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@@
+		)
+	)
+	(text "DNP"
+		(exclude_from_sim no)
+		(at 240.03 96.52 0)
+		(effects
+			(font
+				(size 1.27 1.27)
+				(thickness 0.254)
+				(bold yes)
+				(italic yes)
+				(color 128 77 0 1)
+			)
+		)
+	)
+	(text "DNP"
+		(exclude_from_sim no)
+		(at 240.03 78.74 0)
+		(effects
+			(font
+				(size 1.27 1.27)
+				(thickness 0.254)
+				(bold yes)
+				(italic yes)
+				(color 128 77 0 1)
+			)
 		)
 	)
@@
 	(wire
 		(pts
+			(xy 161.29 138.43) (xy 166.37 138.43)
+		)
+		(stroke
+			(width 0)
+			(type default)
+		)
+	)
+	(wire
+		(pts
 			(xy 34.29 127) (xy 34.29 124.46)
 		)
@@
 		(pts
 			(xy 231.14 99.06) (xy 220.98 99.06)
+		)
+		(stroke
+			(width 0)
+			(type default)
+		)
+	)
+	(wire
+		(pts
+			(xy 161.29 140.97) (xy 161.29 138.43)
 		)
 		(stroke
@@
 		(on_board yes)
 		(dnp no)
-		(fields_autoplaced yes)
 		(property "Reference" "BT1"
-			(at 25.4 36.2584 0)
+			(at 24.13 35.56 0)
 			(effects
 				(font
@@
 		)
 		(property "Value" "18650"
-			(at 25.4 38.7984 0)
+			(at 24.13 38.1 0)
 			(effects
 				(font
@@
 			)
 		)
-		(property "Footprint" ""
+		(property "Footprint" "Wisflow:BatteryHolder_MPD_BK-18650-PC2"
 			(at 21.59 37.846 90)
 			(effects
@@
 			)
 		)
+		(property "JLCPCB" "C19184084"
+			(at 26.67 40.64 0)
+			(effects
+				(font
+					(size 0.762 0.762)
+					(italic yes)
+				)
+			)
+		)
 		(pin "2"
 		)
@@
 		(unit 1)
 		(exclude_from_sim no)
-		(in_bom yes)
+		(in_bom no)
 		(on_board yes)
 		(dnp no)
@@
 			)
 		)
-		(property "Footprint" "Diode_SMD:D_SMA"
+		(property "Footprint" "Connector_JST:JST_EH_S2B-EH_1x02_P2.50mm_Horizontal"
 			(at 40.64 35.56 0)
 			(effects
@@
 	)
 	(symbol
+		(lib_id "power:GND")
+		(at 161.29 140.97 0)
+		(unit 1)
+		(exclude_from_sim no)
+		(in_bom yes)
+		(on_board yes)
+		(dnp no)
+		(property "Reference" "#PWR0111"
+			(at 161.29 147.32 0)
+			(effects
+				(font
+					(size 1.27 1.27)
+				)
+				(hide yes)
+			)
+		)
+		(property "Value" "GND"
+			(at 161.29 144.78 0)
+			(effects
+				(font
+					(size 1.27 1.27)
+				)
+			)
+		)
+		(property "Footprint" ""
+			(at 161.29 140.97 0)
+			(effects
+				(font
+					(size 1.27 1.27)
+				)
+				(hide yes)
+			)
+		)
+		(property "Datasheet" ""
+			(at 161.29 140.97 0)
+			(effects
+				(font
+					(size 1.27 1.27)
+				)
+				(hide yes)
+			)
+		)
+		(property "Description" "Power symbol creates a global label with name \"GND\" , ground"
+			(at 161.29 140.97 0)
+			(effects
+				(font
+					(size 1.27 1.27)
+				)
+				(hide yes)
+			)
+		)
+		(pin "1"
+		)
+		(instances
+			(project "valve-controller_v1.0"
+				(path "/f4047b92-8fb3-4a02-b3b3-070ec973e913"
+					(reference "#PWR0111")
+					(unit 1)
+				)
+			)
+		)
+	)
+	(symbol
 		(lib_id "power:+BATT")
 		(at 35.56 107.95 0)
@@
 	)
 	(symbol
-		(lib_id "Connector_Generic:Conn_01x02")
-		(at 171.45 133.35 0)
+		(lib_id "Connector_Generic:Conn_01x03")
+		(at 171.45 135.89 0)
 		(unit 1)
 		(exclude_from_sim no)
@@
 		)
 		(property "Value" "Debug"
-			(at 173.99 134.62 90)
-			(effects
-				(font
-					(size 1.27 1.27)
-				)
-			)
-		)
-		(property "Footprint" "Connector_PinHeader_2.54mm:PinHeader_1x02_P2.54mm_Vertical"
-			(at 171.45 133.35 0)
+			(at 173.99 135.89 90)
+			(effects
+				(font
+					(size 1.27 1.27)
+				)
+			)
+		)
+		(property "Footprint" "Connector_PinHeader_2.54mm:PinHeader_1x03_P2.54mm_Vertical"
+			(at 171.45 135.89 0)
 			(effects
 				(font
@@
 		)
 		(property "Datasheet" "~"
-			(at 171.45 133.35 0)
-			(effects
-				(font
-					(size 1.27 1.27)
-				)
-				(hide yes)
-			)
-		)
-		(property "Description" "Generic connector, single row, 01x02, script generated (kicad-library-utils/schlib/autogen/connector/)"
-			(at 171.45 133.35 0)
+			(at 171.45 135.89 0)
+			(effects
+				(font
+					(size 1.27 1.27)
+				)
+				(hide yes)
+			)
+		)
+		(property "Description" "Generic connector, single row, 01x03, script generated (kicad-library-utils/schlib/autogen/connector/)"
+			(at 171.45 135.89 0)
 			(effects
 				(font
@@
 		)
 		(pin "2"
+		)
+		(pin "3"
 		)
 		(instances
@@
 		(unit 1)
 		(exclude_from_sim no)
-		(in_bom yes)
-		(on_board yes)
-		(dnp no)
+		(in_bom no)
+		(on_board yes)
+		(dnp no)
