File: valve_controller_v1/valve-controller_v1.0.kicad_sch (KiCad schematic)
At the start: 9 parts, among them J1 Solar Panel, J2 Solenoid #1,2 Output, J3 Solenoid #3,4 Output, J6 Debug

Commit message: Routed PCB and added 3D models
Routed the entire PCB
Added 3D Models for the RAK module and Battery Holder
Improved Silkscreen
Parts:
- removed H1, H2, H3, H4: MountingHole, MountingHole:MountingHole_2.2mm_M2, symbol Mechanical:MountingHole
Connections:
- net Valve Driver/S1_O1: now also J2.2 (Pin_2); no longer J2.1 (Pin_1)
- net Valve Driver/S1_O2: now also J2.1 (Pin_1); no longer J2.2 (Pin_2)
- net Valve Driver/S2_O1: now also J2.4 (Pin_4); no longer J2.3 (Pin_3)
- net Valve Driver/S2_O2: now also J2.3 (Pin_3); no longer J2.4 (Pin_4)
- net Valve Driver/S3_O1: now also J3.2 (Pin_2); no longer J3.1 (Pin_1)
- net Valve Driver/S3_O2: now also J3.1 (Pin_1); no longer J3.2 (Pin_2)
- net Valve Driver/S4_O1: now also J3.4 (Pin_4); no longer J3.3 (Pin_3)
- net Valve Driver/S4_O2: now also J3.3 (Pin_3); no longer J3.4 (Pin_4)
Other:
- added sheet Mechanical and Others (mechanical_and_others.kicad_sch)

Commit message: Created output connector footprint
Created output connector footprint based on the datasheet (Added both parts of the connector, the one soldered to the PCB and the oen that is connected to it)
Added 3D models of both parts and assigned them to the footprint
Relocated the connectors to avoid colission with other components
Rerouted the connectors
Parts:
- J2, J3: footprint Connector_Phoenix_MSTB:PhoenixContact_MSTBA_2,5_4-G-5,08_1x04_P5.08mm_Horizontal -> Wisflow:2EDGRM-5.08-04P
Changed lines of the file:
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@@
 			)
 		)
-		(property "Footprint" "Connector_Phoenix_MSTB:PhoenixContact_MSTBA_2,5_4-G-5,08_1x04_P5.08mm_Horizontal"
+		(property "Footprint" "Wisflow:2EDGRM-5.08-04P"
 			(at 236.22 81.28 0)
 			(effects
@@
 			)
 		)
-		(property "Footprint" "Connector_Phoenix_MSTB:PhoenixContact_MSTBA_2,5_4-G-5,08_1x04_P5.08mm_Horizontal"
+		(property "Footprint" "Wisflow:2EDGRM-5.08-04P"
 			(at 236.22 99.06 0)
 			(effects

Commit message: Final corrections for manufacturing
Created new condenser footprint to better represent the actual position
Created new voltage selector ip switch footprint
Selected bigger footprint for R19 (was 1206 now is 2512 as in the legacy version)
Corrected D5 footprint (was SOD-123 now is SMA)
Parts:
- J1: footprint Connector_JST:JST_EH_S2B-EH_1x02_P2.50mm_Horizontal -> Connector_JST:JST_PH_S2B-PH-SM4-TB_1x02-1MP_P2.00mm_Horizontal
- J6: now left out of the parts list
Changed lines of the file:
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@@
 			)
 		)
-		(property "Footprint" "Connector_JST:JST_EH_S2B-EH_1x02_P2.50mm_Horizontal"
+		(property "Footprint" "Connector_JST:JST_PH_S2B-PH-SM4-TB_1x02-1MP_P2.00mm_Horizontal"
 			(at 40.64 35.56 0)
 			(effects
@@
 		(unit 1)
 		(exclude_from_sim no)
-		(in_bom yes)
-		(on_board yes)
-		(dnp no)
+		(in_bom no)
+		(on_board yes)
+		(dnp no)

Commit message: Added user LED
Added missing user LED. (This LED was present in V0.3c but is missin gin V1.0)
Connections:
- net VCC renamed V_{SOLAR}
Other:
- sheet Power ports: added V_{SOLAR}; removed none
