File: valve_controller_v1/mcu.kicad_sch (KiCad schematic)
At the start: 12 parts, among them J5 Debug & Program, SW2 Reset, SW3 Boot Selector, U4 RAK3172-xx-9-SM-xI

Commit message: Assigned footprints
Assigned footprints
Selected JLCPCB part numbers and searched for alternatives for some components (diodes, transistors)
Imported previos footprint library
Parts:
- SW2: footprint TestPoint:TestPoint_Pad_D1.0mm -> Button_Switch_SMD:SW_SPST_B3U-1000P
- SW3: footprint TestPoint:TestPoint_Pad_D1.0mm -> Button_Switch_SMD:SW_SPDT_PCM12; JLCPCB (none) -> C145854
Changed lines of the file:
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@@
 			)
 		)
-		(property "Footprint" "TestPoint:TestPoint_Pad_D1.0mm"
+		(property "Footprint" "Button_Switch_SMD:SW_SPDT_PCM12"
 			(at 135.89 73.66 0)
 			(effects
@@
 				)
 				(hide yes)
+			)
+		)
+		(property "JLCPCB" "C145854"
+			(at 135.89 81.28 0)
+			(effects
+				(font
+					(size 0.762 0.762)
+					(italic yes)
+				)
 			)
 		)
@@
 			)
 		)
-		(property "Footprint" "TestPoint:TestPoint_Pad_D1.0mm"
+		(property "Footprint" "Button_Switch_SMD:SW_SPST_B3U-1000P"
 			(at 124.46 41.91 0)
 			(effects

Commit message: Basic routing (block level)
Creation of switches footprint
Definition of manufacturing rules
Basic floorplan and layout (routing) of every block
Parts:
- SW3: footprint Button_Switch_SMD:SW_SPDT_PCM12 -> Wisflow:K3-1290S-E1
Connections:
- net RAK_DBG_RX: no longer U4.4 (PB6/UART1_TX)
- new net RAK_DBG_TX: U4.4 (PB6/UART1_TX)
Changed lines of the file:
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@@
+		)
+	)
+	(hierarchical_label "RAK_DBG_RX"
+		(shape input)
+		(at 55.88 142.24 0)
+		(effects
+			(font
+				(size 1.27 1.27)
+			)
+			(justify left)
 		)
 	)
 	(hierarchical_label "RAK_DBG_TX"
-		(shape input)
-		(at 55.88 142.24 0)
-		(effects
-			(font
-				(size 1.27 1.27)
-			)
-			(justify left)
-		)
-	)
-	(hierarchical_label "RAK_DBG_RX"
 		(shape input)
 		(at 55.88 139.7 0)
@@
 			)
 		)
-		(property "Footprint" "Button_Switch_SMD:SW_SPDT_PCM12"
+		(property "Footprint" "Wisflow:K3-1290S-E1"
 			(at 135.89 73.66 0)
 			(effects
