File: valve_controller_v1/mcu.kicad_sch (KiCad schematic)
At the start: 12 parts, among them J5 Debug & Program, SW2 Reset, SW3 Boot Selector, U4 RAK3172-xx-9-SM-xI

Commit message: Routed PCB and added 3D models
Routed the entire PCB
Added 3D Models for the RAK module and Battery Holder
Improved Silkscreen
Parts:
- removed TP10: BAT_MON, TestPoint:TestPoint_Pad_D1.0mm, symbol Connector:TestPoint
- removed TP9: ~{BAT_MON_EN}, TestPoint:TestPoint_Pad_D1.0mm, symbol Connector:TestPoint
- renumbered TP11 to TP9
Connections:
- net BAT_MON: now also U4.31 (PB4/PIN_A1); no longer U4.32 (PB3/PIN_A0)
- net RAK_CTRL_S1_I1: now also U4.19 (PA8); no longer U4.16 (PA4/~{SPI1_SS})
- net RAK_CTRL_S1_I2: now also U4.20 (PA9); no longer U4.15 (PA5/SPI1_CLK)
- net RAK_CTRL_S2_I1: now also U4.15 (PA5/SPI1_CLK); no longer U4.14 (PA6/SPI1_MISO)
- net RAK_CTRL_S2_I2: now also U4.16 (PA4/~{SPI1_SS}); no longer U4.13 (PA7/SPI1_MOSI)
- net RAK_CTRL_S3_I1: now also U4.13 (PA7/SPI1_MOSI); no longer U4.6 (PA1)
- net RAK_CTRL_S3_I2: now also U4.14 (PA6/SPI1_MISO); no longer U4.19 (PA8)
- net RAK_CTRL_S4_I1: now also U4.10 (PA11/SDA); no longer U4.20 (PA9)
- net RAK_CTRL_S4_I2: now also U4.9 (PA12/SCL); no longer U4.25 (PA10/PIN_A3)
- net ~{BAT_MON_EN}: now also U4.32 (PB3/PIN_A0); no longer U4.26 (PB2/PIN_A2)
Changed lines of the file:
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@@
-	)
-	(no_connect
-		(at 88.9 69.85)
-	)
-	(no_connect
-		(at 48.26 44.45)
 	)
 	(no_connect
@@
 	)
 	(no_connect
-		(at 88.9 67.31)
+		(at 88.9 64.77)
 	)
 	(no_connect
 		(at 48.26 46.99)
 	)
+	(no_connect
+		(at 48.26 39.37)
+	)
+	(no_connect
+		(at 88.9 41.91)
+	)
 	(wire
 		(pts
@@
 	(wire
 		(pts
+			(xy 88.9 69.85) (xy 106.68 69.85)
+		)
+		(stroke
+			(width 0)
+			(type default)
+		)
+	)
+	(wire
+		(pts
 			(xy 88.9 62.23) (xy 106.68 62.23)
 		)
@@
 	(wire
 		(pts
-			(xy 168.91 76.2) (xy 156.21 76.2)
-		)
-		(stroke
-			(width 0)
-			(type default)
-		)
-	)
-	(wire
-		(pts
 			(xy 160.02 27.94) (xy 160.02 30.48)
 		)
@@
 	(wire
 		(pts
-			(xy 88.9 64.77) (xy 106.68 64.77)
-		)
-		(stroke
-			(width 0)
-			(type default)
-		)
-	)
-	(wire
-		(pts
 			(xy 30.48 34.29) (xy 48.26 34.29)
 		)
@@
 	(wire
 		(pts
-			(xy 168.91 78.74) (xy 156.21 78.74)
-		)
-		(stroke
-			(width 0)
-			(type default)
-		)
-	)
-	(wire
-		(pts
 			(xy 96.52 127) (xy 77.47 127)
 		)
@@
 	(wire
 		(pts
+			(xy 88.9 67.31) (xy 106.68 67.31)
+		)
+		(stroke
+			(width 0)
+			(type default)
+		)
+	)
+	(wire
+		(pts
 			(xy 30.48 41.91) (xy 48.26 41.91)
 		)
@@
 	(wire
 		(pts
-			(xy 30.48 39.37) (xy 48.26 39.37)
-		)
-		(stroke
-			(width 0)
-			(type default)
-		)
-	)
-	(wire
-		(pts
-			(xy 88.9 41.91) (xy 106.68 41.91)
+			(xy 30.48 44.45) (xy 48.26 44.45)
 		)
 		(stroke
@@
 	)
 	(label "RAK_CTRL_S4_I1"
+		(at 106.68 67.31 180)
+		(effects
+			(font
+				(size 1.27 1.27)
+			)
+			(justify right bottom)
+		)
+	)
+	(label "RAK_CTRL_S1_I2"
 		(at 106.68 62.23 180)
 		(effects
@@
 		)
 	)
-	(label "RAK_CTRL_S1_I2"
-		(at 106.68 52.07 180)
-		(effects
-			(font
-				(size 1.27 1.27)
-			)
-			(justify right bottom)
-		)
-	)
 	(label "RAK_CTRL_S4_I2"
-		(at 106.68 64.77 180)
+		(at 106.68 69.85 180)
 		(effects
 			(font
@@
 	)
 	(label "RAK_CTRL_S3_I1"
-		(at 106.68 41.91 180)
+		(at 106.68 57.15 180)
 		(effects
 			(font
@@
 	)
 	(label "BAT_MON"
-		(at 30.48 41.91 0)
+		(at 30.48 44.45 0)
 		(effects
 			(font
@@
 	)
 	(label "RAK_CTRL_S1_I1"
-		(at 106.68 49.53 180)
+		(at 106.68 59.69 180)
 		(effects
 			(font
@@
 	)
 	(label "~{BAT_MON_EN}"
-		(at 30.48 39.37 0)
+		(at 30.48 41.91 0)
 		(effects
 			(font
@@
 	)
 	(label "RAK_CTRL_S3_I2"
-		(at 106.68 59.69 180)
+		(at 106.68 54.61 180)
 		(effects
 			(font
@@
 	)
 	(label "RAK_CTRL_S2_I1"
-		(at 106.68 54.61 180)
+		(at 106.68 52.07 180)
 		(effects
 			(font
@@
 		)
 	)
-	(label "~{BAT_MON_EN}"
-		(at 156.21 76.2 0)
-		(effects
-			(font
-				(size 1.27 1.27)
-			)
-			(justify left bottom)
-		)
-	)
 	(label "RAK_UART_RX"
 		(at 39.37 111.76 0)
@@
 	)
 	(label "RAK_CTRL_S2_I2"
-		(at 106.68 57.15 180)
+		(at 106.68 49.53 180)
 		(effects
 			(font
@@
 			)
 			(justify right bottom)
-		)
-	)
-	(label "BAT_MON"
-		(at 156.21 78.74 0)
-		(effects
-			(font
-				(size 1.27 1.27)
-			)
-			(justify left bottom)
 		)
 	)
@@
 			)
 			(justify left)
-		)
-	)
-	(symbol
-		(lib_id "Connector:TestPoint")
-		(at 168.91 78.74 270)
-		(unit 1)
-		(exclude_from_sim no)
-		(in_bom yes)
-		(on_board yes)
-		(dnp no)
-		(property "Reference" "TP10"
-			(at 173.99 77.4699 90)
-			(effects
-				(font
-					(size 1.27 1.27)
-				)
-				(justify left)
-				(hide yes)
-			)
-		)
-		(property "Value" "BAT_MON"
-			(at 173.99 78.74 90)
-			(effects
-				(font
-					(size 1.27 1.27)
-				)
-				(justify left)
-			)
-		)
-		(property "Footprint" "TestPoint:TestPoint_Pad_D1.0mm"
-			(at 168.91 83.82 0)
-			(effects
-				(font
-					(size 1.27 1.27)
-				)
-				(hide yes)
-			)
-		)
-		(property "Datasheet" "~"
-			(at 168.91 83.82 0)
-			(effects
-				(font
-					(size 1.27 1.27)
-				)
-				(hide yes)
-			)
-		)
-		(property "Description" "test point"
-			(at 168.91 78.74 0)
-			(effects
-				(font
-					(size 1.27 1.27)
-				)
-				(hide yes)
-			)
-		)
-		(pin "1"
-		)
-		(instances
-			(project "valve-controller_v1.0"
-				(path "/f4047b92-8fb3-4a02-b3b3-070ec973e913/71e93b2c-65ce-4650-9976-c707bec3d8ef"
-					(reference "TP10")
-					(unit 1)
-				)
-			)
-		)
-	)
-	(symbol
-		(lib_id "Connector:TestPoint")
-		(at 168.91 76.2 270)
-		(unit 1)
-		(exclude_from_sim no)
-		(in_bom yes)
-		(on_board yes)
-		(dnp no)
-		(property "Reference" "TP9"
-			(at 173.99 74.9299 90)
-			(effects
-				(font
-					(size 1.27 1.27)
-				)
-				(justify left)
-				(hide yes)
-			)
-		)
-		(property "Value" "~{BAT_MON_EN}"
-			(at 173.99 76.2 90)
-			(effects
-				(font
-					(size 1.27 1.27)
-				)
-				(justify left)
-			)
-		)
-		(property "Footprint" "TestPoint:TestPoint_Pad_D1.0mm"
-			(at 168.91 81.28 0)
-			(effects
-				(font
-					(size 1.27 1.27)
-				)
-				(hide yes)
-			)
-		)
-		(property "Datasheet" "~"
-			(at 168.91 81.28 0)
-			(effects
-				(font
-					(size 1.27 1.27)
-				)
-				(hide yes)
-			)
-		)
-		(property "Description" "test point"
-			(at 168.91 76.2 0)
-			(effects
-				(font
-					(size 1.27 1.27)
-				)
-				(hide yes)
-			)
-		)
-		(pin "1"
-		)
-		(instances
-			(project "valve-controller_v1.0"
-				(path "/f4047b92-8fb3-4a02-b3b3-070ec973e913/71e93b2c-65ce-4650-9976-c707bec3d8ef"
-					(reference "TP9")
-					(unit 1)
-				)
-			)
 		)
 	)
@@
 		(on_board yes)
 		(dnp no)
-		(property "Reference" "TP11"
+		(property "Reference" "TP9"
 			(at 173.99 80.0099 90)
 			(effects
@@
 			(project "valve-controller_v1.0"
 				(path "/f4047b92-8fb3-4a02-b3b3-070ec973e913/71e93b2c-65ce-4650-9976-c707bec3d8ef"
-					(reference "TP11")
+					(reference "TP9")
 					(unit 1)
 				)

Commit message: Final corrections for manufacturing
Created new condenser footprint to better represent the actual position
Created new voltage selector ip switch footprint
Selected bigger footprint for R19 (was 1206 now is 2512 as in the legacy version)
Corrected D5 footprint (was SOD-123 now is SMA)
Parts:
- JP1, TP9: now left out of the parts list
Changed lines of the file:
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@@
 		(unit 1)
 		(exclude_from_sim no)
-		(in_bom yes)
+		(in_bom no)
 		(on_board yes)
 		(dnp no)
@@
 		(unit 1)
 		(exclude_from_sim no)
-		(in_bom yes)
-		(on_board yes)
-		(dnp no)
+		(in_bom no)
+		(on_board yes)
+		(dnp no)

Commit message: Added user LED
Added missing user LED. (This LED was present in V0.3c but is missin gin V1.0)
Parts:
- added D6: Blue, LED_SMD:LED_0603_1608Metric, symbol Device:LED_Small_Filled
- added R24: 1k, Resistor_SMD:R_0603_1608Metric, symbol Device:R_Small
Connections:
- net GND: now also D6.1 (K)
- net RAK_LED: now reaches U4.25 (PA10/PIN_A3)
- net RAK_LED: now also R24.1
- new net: D6.2 (A), R24.2
- no-connect marks 7 -> 6
Other:
- note added: "Uer LED"
