File: valve_controller_v1/power.kicad_sch (KiCad schematic)
At the start: 26 parts, among them Q1 DMG3415UQ-7, Q2 BSD235C, SW1 XKB5858, U1 BQ21040DBV, U2 XC6220B331MR

Commit message: Assigned footprints
Assigned footprints
Selected JLCPCB part numbers and searched for alternatives for some components (diodes, transistors)
Imported previos footprint library
Parts:
- removed Q2: BSD235C, Package_TO_SOT_SMD:SOT-363_SC-70-6, symbol Transistor_FET:BSD235C
- added Q3: AP2003, Package_TO_SOT_SMD:TSOT-23-6, symbol Transistor_FET:DMC2053UVT
- D1, D2, D3: footprint Diode_SMD:D_SC-80 -> Diode_SMD:D_SOD-123; JLCPCB (none) -> C8598
- Q1: value DMG3415UQ-7 -> AO3401A; footprint (none) -> Package_TO_SOT_SMD:SOT-23; JLCPCB (none) -> C15127
- SW1: footprint TestPoint:TestPoint_Pad_D1.0mm -> Button_Switch_SMD:Panasonic_EVQPUJ_EVQPUA; JLCPCB (none) -> C780036
- U1: JLCPCB (none) -> C202311
- U2: JLCPCB (none) -> C86534
Connections:
- net +BATT: now also Q3.2 (S)
- net GND: now also Q3.5 (S)
- net ~{BAT_MON_EN}: now also Q3.1 (G)
- net at R6.2: now also Q3.3 (G), Q3.6 (D)
- net at R7.1: now also Q3.4 (D)
Other:
- note removed: "JLCPCB: C780036"

Commit message: Basic routing (block level)
Creation of switches footprint
Definition of manufacturing rules
Basic floorplan and layout (routing) of every block
Parts:
- SW1: footprint Button_Switch_SMD:Panasonic_EVQPUJ_EVQPUA -> Wisflow:XKB5858-X-F-75
Changed lines of the file:
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@@
 			)
 		)
-		(property "Footprint" "Button_Switch_SMD:Panasonic_EVQPUJ_EVQPUA"
+		(property "Footprint" "Wisflow:XKB5858-X-F-75"
 			(at 99.06 53.34 0)
 			(effects
