File: valve_controller_v1/power.kicad_sch (KiCad schematic)
At the start: 26 parts, among them Q1 AO3401A, Q3 AP2003, SW1 XKB5858, U1 BQ21040DBV, U2 XC6220B331MR

Commit message: Final corrections for manufacturing
Created new condenser footprint to better represent the actual position
Created new voltage selector ip switch footprint
Selected bigger footprint for R19 (was 1206 now is 2512 as in the legacy version)
Corrected D5 footprint (was SOD-123 now is SMA)
Parts:
- TP1, TP2, TP3, TP4, TP5, TP6: now left out of the parts list
Changed lines of the file:
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@@
 		(unit 1)
 		(exclude_from_sim no)
-		(in_bom yes)
+		(in_bom no)
 		(on_board yes)
 		(dnp no)
@@
 		(unit 1)
 		(exclude_from_sim no)
-		(in_bom yes)
+		(in_bom no)
 		(on_board yes)
 		(dnp no)
@@
 		(unit 1)
 		(exclude_from_sim no)
-		(in_bom yes)
+		(in_bom no)
 		(on_board yes)
 		(dnp no)
@@
 		(unit 1)
 		(exclude_from_sim no)
-		(in_bom yes)
+		(in_bom no)
 		(on_board yes)
 		(dnp no)
@@
 		(unit 1)
 		(exclude_from_sim no)
-		(in_bom yes)
+		(in_bom no)
 		(on_board yes)
 		(dnp no)
@@
 		(unit 1)
 		(exclude_from_sim no)
-		(in_bom yes)
-		(on_board yes)
-		(dnp no)
+		(in_bom no)
+		(on_board yes)
+		(dnp no)

Commit message: Added user LED
Added missing user LED. (This LED was present in V0.3c but is missin gin V1.0)
Connections:
- net VCC: now also C2.1, R3.1, U2.1 (VIN); no longer D3.2 (A)
- net VDD: no longer C2.1, R3.1, U2.1 (VIN)
- new net V_{SOLAR}: D3.2 (A)
