File: valve_controller_v1/step_up.kicad_sch (KiCad schematic)
At the start: 17 parts, among them SW4 Voltage Selector, U5 LT218, U6 LMR62421XMF

Commit message: Assigned footprints
Assigned footprints
Selected JLCPCB part numbers and searched for alternatives for some components (diodes, transistors)
Imported previos footprint library
Parts:
- C12: now left out of the parts list
- D5: JLCPCB (none) -> C8678
- L1: value L_Small -> 6.8uH; footprint (none) -> Inductor_SMD:L_Sunlord_SWPA5040S; JLCPCB (none) -> C36411
- R19: footprint Resistor_SMD:R_0603_1608Metric -> Resistor_SMD:R_1206_3216Metric
- SW4: JLCPCB (none) -> C5439234
- U5: footprint (none) -> Package_SO:SO-4_4.4x4.3mm_P2.54mm; JLCPCB (none) -> C2691608
- U6: JLCPCB (none) -> C544413
Other:
- note added: "DNP"
Changed lines of the file:
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@@
+		)
+	)
+	(text "DNP"
+		(exclude_from_sim no)
+		(at 163.83 36.83 0)
+		(effects
+			(font
+				(size 1.27 1.27)
+				(thickness 0.254)
+				(bold yes)
+				(italic yes)
+				(color 128 77 0 1)
+			)
 		)
 	)
@@
 			)
 		)
-		(property "Footprint" "Resistor_SMD:R_0603_1608Metric"
+		(property "Footprint" "Resistor_SMD:R_1206_3216Metric"
 			(at 160.02 29.21 0)
 			(effects
@@
 		(dnp no)
 		(property "Reference" "SW4"
+			(at 127 46.99 0)
+			(effects
+				(font
+					(size 1.27 1.27)
+				)
+			)
+		)
+		(property "Value" "Voltage Selector"
 			(at 116.84 46.99 0)
-			(effects
-				(font
-					(size 1.27 1.27)
-				)
-			)
-		)
-		(property "Value" "Voltage Selector"
-			(at 127 46.99 0)
 			(effects
 				(font
@@
 				)
 				(hide yes)
+			)
+		)
+		(property "JLCPCB" "C5439234"
+			(at 127 52.07 90)
+			(effects
+				(font
+					(size 0.762 0.762)
+					(italic yes)
+				)
 			)
 		)
@@
 			)
 		)
+		(property "JLCPCB" "C544413"
+			(at 85.09 62.23 0)
+			(effects
+				(font
+					(size 0.762 0.762)
+					(italic yes)
+				)
+			)
+		)
 		(pin "5"
 		)
@@
 			)
 		)
-		(property "Footprint" ""
+		(property "Footprint" "Package_SO:SO-4_4.4x4.3mm_P2.54mm"
 			(at 50.8 44.45 0)
 			(effects
@@
 				)
 				(hide yes)
+			)
+		)
+		(property "JLCPCB" "C2691608"
+			(at 50.8 52.07 0)
+			(effects
+				(font
+					(size 0.762 0.762)
+					(italic yes)
+				)
 			)
 		)
@@
 		(on_board yes)
 		(dnp no)
-		(fields_autoplaced yes)
 		(property "Reference" "L1"
 			(at 81.28 36.83 90)
@@
 			)
 		)
-		(property "Value" "L_Small"
+		(property "Value" "6.8uH"
 			(at 81.28 39.37 90)
 			(effects
@@
 			)
 		)
-		(property "Footprint" ""
+		(property "Footprint" "Inductor_SMD:L_Sunlord_SWPA5040S"
 			(at 81.28 41.91 0)
 			(effects
@@
 				)
 				(hide yes)
+			)
+		)
+		(property "JLCPCB" "C36411"
+			(at 81.28 43.18 90)
+			(effects
+				(font
+					(size 0.762 0.762)
+					(italic yes)
+				)
 			)
 		)
@@
 		(unit 1)
 		(exclude_from_sim no)
-		(in_bom yes)
+		(in_bom no)
 		(on_board yes)
 		(dnp no)
@@
 			)
 		)
+		(property "JLCPCB" "C8678"
+			(at 96.52 46.99 0)
+			(effects
+				(font
+					(size 0.762 0.762)
+					(italic yes)
+				)
+			)
+		)

Commit message: Basic routing (block level)
Creation of switches footprint
Definition of manufacturing rules
Basic floorplan and layout (routing) of every block
Parts:
- SW4: footprint TestPoint:TestPoint_Pad_D1.0mm -> Package_SO:SO-4_4.4x4.3mm_P2.54mm
Changed lines of the file:
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@@
 			)
 		)
-		(property "Footprint" "TestPoint:TestPoint_Pad_D1.0mm"
+		(property "Footprint" "Package_SO:SO-4_4.4x4.3mm_P2.54mm"
 			(at 123.19 46.99 0)
 			(effects
