File: valve_controller_v1/valve-controller_v1.0.kicad_pcb (KiCad board)
At the start: 2 copper layers, 77 parts, among them J1 Solar Panel, J2 Solenoid #1,2 Output, J3 Solenoid #3,4 Output, J4 USB_C_Receptacle_USB2.0_16P, J5 Debug & Program, J6 Debug, Q2 BSD235C, SW1 XKB5858, SW2 Reset, SW3 Boot Selector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

Commit message: Assigned footprints
Assigned footprints
Selected JLCPCB part numbers and searched for alternatives for some components (diodes, transistors)
Imported previos footprint library
Parts:
- added BT1: 18650, Wisflow:BatteryHolder_MPD_BK-18650-PC2, F.Cu at (-110.5, 51.3)
- added L1: 6.8uH, Inductor_SMD:L_Sunlord_SWPA5040S, F.Cu at (-347.2, -46.1)
- added Q1: AO3401A, Package_TO_SOT_SMD:SOT-23, F.Cu at (-147.7, -66.0)
- added Q3: AP2003, Package_TO_SOT_SMD:TSOT-23-6, F.Cu at (-134.7, -28.3)
- added U5: LT218, Package_SO:SO-4_4.4x4.3mm_P2.54mm, F.Cu at (-337.3, -58.9)
- D1, D2, D3: footprint Diode_SMD:D_SC-80 -> Diode_SMD:D_SOD-123
- J1: footprint Diode_SMD:D_SMA -> Connector_JST:JST_EH_S2B-EH_1x02_P2.50mm_Horizontal
- J6: footprint Connector_PinHeader_2.54mm:PinHeader_1x02_P2.54mm_Vertical -> Connector_PinHeader_2.54mm:PinHeader_1x03_P2.54mm_Vertical
- R19: footprint Resistor_SMD:R_0603_1608Metric -> Resistor_SMD:R_1206_3216Metric
- SW1, SW3: footprint TestPoint:TestPoint_Pad_D1.0mm -> Button_Switch_SMD:Panasonic_EVQPUJ_EVQPUA
- SW2: footprint TestPoint:TestPoint_Pad_D1.0mm -> Button_Switch_SMD:SW_SPST_B3U-1000P
- moved J6 19.6 mm to (-219.8, -137.9), turned to 90 degrees
- moved SW2 11.1 mm to (-386.0, -163.6)
- moved C8 9.50 mm to (-385.2, -166.5), turned to 180 degrees
- moved JP1 8.69 mm to (-394.6, -147.2)
- moved R12 8.31 mm to (-385.1, -160.8)
- moved SW3 3.86 mm to (-399.3, -148.2), turned to 90 degrees
Connections:
- R6 pad 2: Net-(Q2A-DN) -> Net-(Q3A-D)
- R7 pad 1: Net-(Q2B-DP) -> Net-(Q3B-D)

Commit message: Basic routing (block level)
Creation of switches footprint
Definition of manufacturing rules
Basic floorplan and layout (routing) of every block
Parts:
- removed Q2: BSD235C, Package_TO_SOT_SMD:SOT-363_SC-70-6
- SW1: footprint Button_Switch_SMD:Panasonic_EVQPUJ_EVQPUA -> Wisflow:XKB5858-X-F-75
- SW3: footprint Button_Switch_SMD:Panasonic_EVQPUJ_EVQPUA -> Wisflow:K3-1290S-E1
- SW4: footprint TestPoint:TestPoint_Pad_D1.0mm -> Package_SO:SO-4_4.4x4.3mm_P2.54mm
- moved TP11 237.7 mm to (-182.4, -51.1)
- moved TP9 237.7 mm to (-182.4, -57.2)
- moved TP10 237.7 mm to (-182.4, -54.1)
- moved C8 169.3 mm to (-216.5, -152.6), turned to -90 degrees
- moved R12 167.0 mm to (-218.2, -152.6), turned to 90 degrees
- moved J5 166.3 mm to (-230.4, -152.6)
- moved SW3 165.3 mm to (-234.0, -145.3), turned to 0 degrees
- moved SW2 164.5 mm to (-221.8, -152.6)
- moved JP1 159.2 mm to (-235.5, -152.6), turned to 90 degrees
- moved C7 137.0 mm to (-257.8, -156.2)
- moved C6 136.5 mm to (-257.8, -157.9)
- moved BT1 106.7 mm to (-156.6, -44.9)
- moved R6 103.8 mm to (-230.3, -55.7), turned to 180 degrees
- moved R5 102.2 mm to (-230.3, -57.5), turned to 180 degrees
- moved R8 102.0 mm to (-227.5, -52.8), turned to 90 degrees
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Connections:
- J6 pad 1: /MCU/RAK_DBG_RX -> /MCU/RAK_DBG_TX
- U4 pad 4: /MCU/RAK_DBG_RX -> /MCU/RAK_DBG_TX
Routing:
- net GND: track 1.32 -> 19.8 mm, vias 1 -> 13
- net Net-(U6-FB): track 0.00 -> 18.4 mm
- net Net-(D5-K): track 0.00 -> 15.3 mm
- net VDD: track 0.00 -> 15.3 mm
- net Net-(U6-VIN): track 0.00 -> 11.1 mm
- net Net-(Q3A-D): track 0.00 -> 8.27 mm
- net Net-(R13-Pad2): track 0.00 -> 6.85 mm
- net VBUS: track 6.56 -> 0.00 mm
- net Net-(D5-A): track 0.00 -> 5.83 mm
- net /Valve Driver/S2_O1: track 0.00 -> 5.08 mm
- net /Valve Driver/S1_O1: track 0.00 -> 5.08 mm
- net /Valve Driver/S4_O1: track 0.00 -> 5.08 mm
- net /Valve Driver/S3_O1: track 0.00 -> 5.08 mm
- net VCC: track 0.00 -> 4.91 mm
- net /Valve Driver/S4_O2: track 0.00 -> 4.87 mm
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Other:
- copper layers 2 -> 4

Commit message: Corrected power switch footprint
Corrected the footprint (numbering of the pins) according to the EasyEDA footprint model on JLCPCB
Reviewed the boot select footprint pin assignment also
Parts:
- moved C2 413.2 mm to (134.4, -23.4), turned to -90 degrees
- moved C4 411.4 mm to (133.3, -16.5), turned to 180 degrees
- moved SW1 411.3 mm to (130.3, -19.6)
- moved U2 411.2 mm to (133.3, -19.6), turned to -90 degrees
- moved BT1 410.9 mm to (254.3, -40.3)
- moved C10 410.9 mm to (118.0, -47.2)
- moved C11 410.9 mm to (116.1, -51.7)
- moved C13 410.9 mm to (116.8, -54.3)
- moved C6 410.9 mm to (153.0, -153.4)
- moved C7 410.9 mm to (153.0, -151.6)
- moved C9 410.9 mm to (126.6, -50.0)
- moved D4 410.9 mm to (188.0, -78.5)
- moved D5 410.9 mm to (118.3, -50.9)
- moved J1 410.9 mm to (192.1, -27.3)
- moved JP1 410.9 mm to (175.3, -148.0)
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