File: valve_controller_v1/mechanical_and_others.kicad_sch (KiCad schematic)
At the start: 4 parts

Commit message: Added logo and minor footprint location corrections
Added Wisflow Logo on front silkscreen
Added logo, revision and serial number text on the back silkscreen
Added jumper description on the back silkscreen
Corrected battery holder and capacitor location to avoid colision with the case (middle screw boss)
Parts:
- added LG1: ~, Wisflow:WisflowLogo_30mm, symbol Wisflow:WisflowLogo
- added LG2: ~, Wisflow:WisflowLogo_20mm, symbol Wisflow:WisflowLogo
Changed lines of the file:
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@@
+	)
+	(symbol
+		(lib_id "Wisflow:WisflowLogo")
+		(at 55.88 27.94 0)
+		(unit 1)
+		(exclude_from_sim no)
+		(in_bom no)
+		(on_board yes)
+		(dnp no)
+		(property "Reference" "LG1"
+			(at 50.8 24.13 0)
+			(effects
+				(font
+					(size 1.27 1.27)
+				)
+				(justify left)
+			)
+		)
+		(property "Value" "~"
+			(at 55.88 27.94 0)
+			(effects
+				(font
+					(size 1.27 1.27)
+				)
+				(hide yes)
+			)
+		)
+		(property "Footprint" "Wisflow:WisflowLogo_30mm"
+			(at 55.88 27.94 0)
+			(effects
+				(font
+					(size 1.27 1.27)
+				)
+				(hide yes)
+			)
+		)
+		(property "Datasheet" ""
+			(at 55.88 27.94 0)
+			(effects
+				(font
+					(size 1.27 1.27)
+				)
+				(hide yes)
+			)
+		)
+		(property "Description" ""
+			(at 55.88 27.94 0)
+			(effects
+				(font
+					(size 1.27 1.27)
+				)
+				(hide yes)
+			)
+		)
+		(instances
+			(project "valve-controller_v1.0"
+				(path "/f4047b92-8fb3-4a02-b3b3-070ec973e913/e6b8d514-00e8-4e46-870f-fd1d3900ef71"
+					(reference "LG1")
+					(unit 1)
+				)
+			)
+		)
 	)
 	(symbol
@@
 					(unit 1)
 				)
+			)
+		)
+	)
+	(symbol
+		(lib_id "Wisflow:WisflowLogo")
+		(at 55.88 38.1 0)
+		(unit 1)
+		(exclude_from_sim no)
+		(in_bom no)
+		(on_board yes)
+		(dnp no)
+		(property "Reference" "LG2"
+			(at 50.8 34.29 0)
+			(effects
+				(font
+					(size 1.27 1.27)
+				)
+				(justify left)
+			)
+		)
+		(property "Value" "~"
+			(at 55.88 38.1 0)
+			(effects
+				(font
+					(size 1.27 1.27)
+				)
+				(hide yes)
+			)
+		)
+		(property "Footprint" "Wisflow:WisflowLogo_20mm"
+			(at 55.88 38.1 0)
+			(effects
+				(font
+					(size 1.27 1.27)
+				)
+				(hide yes)
+			)
+		)
+		(property "Datasheet" ""
+			(at 55.88 38.1 0)
+			(effects
+				(font
+					(size 1.27 1.27)
+				)
+				(hide yes)
+			)
+		)
+		(property "Description" ""
+			(at 55.88 38.1 0)
+			(effects
+				(font
+					(size 1.27 1.27)
+				)
+				(hide yes)
+			)
+		)
+		(instances
+			(project "valve-controller_v1.0"
+				(path "/f4047b92-8fb3-4a02-b3b3-070ec973e913/e6b8d514-00e8-4e46-870f-fd1d3900ef71"
+					(reference "LG2")
+					(unit 1)
+				)

Commit message: Added user LED
Added missing user LED. (This LED was present in V0.3c but is missin gin V1.0)
Parts:
- LG1, LG2: value ~ -> (none)
